Commit message: use effort controller of ur5

File: jsk_mbzirc_tasks/urdf/husky_with_camera.urdf.xacro (robot description, xacro)
@@ -4,9 +4,9 @@
   <xacro:arg name="kinect_enabled" default="false" />
   <xacro:arg name="gripper_enabled" default="false" />
-  <xacro:include filename="$(find husky_description)/urdf/husky.urdf.xacro" />
-  <xacro:include filename="$(find husky_gazebo)/urdf/husky.gazebo.xacro" />
   <!-- use effor controller -->
   <xacro:arg name="use_position_interface" default="false" />
   <xacro:arg name="use_effort_interface" default="true" />
+  <xacro:include filename="$(find husky_description)/urdf/husky.urdf.xacro" />
+  <xacro:include filename="$(find husky_gazebo)/urdf/husky.gazebo.xacro" />
   <!-- Gazebo plugin for ROS Control -->
   <gazebo>
@@ -16,4 +16,15 @@
   </gazebo>
   <xacro:husky_robot />
+  <xacro:property name="reflect" value="-1" />
+  <!-- Spawn arm -->
+  <xacro:ur5_robot prefix="ur5_arm_" joint_limited="true"/>
+  <!-- Join arm -->
+  <joint name="ur5_arm_base" type="fixed">
+    <parent link="top_plate_link" />
+    <child link="ur5_arm_base_link" />
+    <origin xyz="0.3058 0 0.0065" rpy="0.0 0.0 -1.57" />
+  </joint>
+  <!-- Spawn gripper -->
+  <xacro:pr2_gripper_simple_transmission />
   <xacro:husky_robot_gazebo />
   <!-- Forward facing camera -->

Commit message: add hand-eye camera for task2

File: jsk_mbzirc_tasks/urdf/husky_with_camera.urdf.xacro (robot description, xacro)
@@ -33,3 +33,8 @@
     <origin xyz="-0.3 0.0 0.6" rpy="0 0 0"/>
   </xacro:generic_camera>
+  <!-- Hand eye camera -->
+  <xacro:include filename="$(find hector_sensors_description)/urdf/generic_camera.urdf.xacro" />
+  <xacro:generic_camera name="handeye_camera" parent="r_gripper_tool_frame" ros_topic="image" cam_info_topic="camera_info" update_rate="20" res_x="640" res_y="480" image_format="L8" hfov="90">
+    <origin xyz="-0.10 0.0 0.2" rpy="0 0.785 0"/>
+  </xacro:generic_camera>
 </robot>
