Commit message: added another camera for side view on quadrotor and tf on rviz

File: jsk_mbzirc_tasks/urdf/quadrotor_with_hokyo30lx_and_downward_cam.urdf.xacro (robot description, xacro)
@@ -10,11 +10,18 @@
     <!-- Hokuyo UTM-30LX mounted upside down below the quadrotor body -->
     <xacro:include filename="$(find hector_sensors_description)/urdf/hokuyo_utm30lx.urdf.xacro" />
-    <xacro:hokuyo_utm30lx name="laser0" parent="base_link" ros_topic="scan" update_rate="40" ray_count="1081" min_angle="-135" max_angle="135">
+    <xacro:hokuyo_utm30lx name="laser0" parent="base_link" ros_topic="scan" update_rate="40"
+			  ray_count="1081" min_angle="-135" max_angle="135">
       <origin xyz="0.0 0.0 -0.097" rpy="${M_PI} 0 0"/>
     </xacro:hokuyo_utm30lx>
     <!-- Downward facing camera -->
     <xacro:include filename="$(find hector_sensors_description)/urdf/generic_camera.urdf.xacro" />
-    <xacro:generic_camera name="downward_cam" parent="base_link" ros_topic="camera/image" cam_info_topic="camera/camera_info" update_rate="20" res_x="640" res_y="480" image_format="L8" hfov="100">
+    <xacro:generic_camera name="downward_cam" parent="base_link" ros_topic="camera/image" cam_info_topic="camera/camera_info"
+			  update_rate="20" res_x="640" res_y="480" image_format="L8" hfov="100">
       <origin xyz="0.4 0.0 -0.0" rpy="0 ${M_PI/2} 0"/>
     </xacro:generic_camera>
+    <!-- side facing camera -->
+    <xacro:generic_camera name="side_cam" parent="base_link" ros_topic="camera/image" cam_info_topic="camera/camera_info"
+			  update_rate="20" res_x="640" res_y="480" image_format="L8" hfov="100">
+      <origin xyz="-0.4 0.0 -0.0" rpy="${M_PI} ${M_PI} 0"/>
+    </xacro:generic_camera>
 </robot>

Commit message: move camera to centerand change to wild FOV

File: jsk_mbzirc_tasks/urdf/quadrotor_with_hokyo30lx_and_downward_cam.urdf.xacro (robot description, xacro)
@@ -15,6 +15,6 @@
     <!-- Downward facing camera -->
     <xacro:include filename="$(find hector_sensors_description)/urdf/generic_camera.urdf.xacro" />
-    <xacro:generic_camera name="downward_cam" parent="base_link" ros_topic="camera/image" cam_info_topic="camera/camera_info" update_rate="20" res_x="640" res_y="480" image_format="L8" hfov="100">
-      <origin xyz="0.4 0.0 -0.0" rpy="0 ${M_PI/2} 0"/>
+    <xacro:generic_camera name="downward_cam" parent="base_link" ros_topic="camera/image" cam_info_topic="camera/camera_info" update_rate="20" res_x="640" res_y="480" image_format="L8" hfov="160">
+      <origin xyz="0.0 0.0 -0.2" rpy="0 ${M_PI/2} 0"/>
     </xacro:generic_camera>
 </robot>

Commit message: camera side wards

File: jsk_mbzirc_tasks/urdf/quadrotor_with_hokyo30lx_and_downward_cam.urdf.xacro (robot description, xacro)
@@ -18,3 +18,8 @@
       <origin xyz="0.4 0.0 -0.0" rpy="0 ${M_PI/2} 0"/>
     </xacro:generic_camera>
+    <!-- side facing camera -->
+    <xacro:generic_camera name="side_cam" parent="base_link" ros_topic="camera/image" cam_info_topic="camera/camera_info"
+			    update_rate="20" res_x="640" res_y="480" image_format="L8" hfov="100">
+      <origin xyz="-0.4 0.0 -0.0" rpy="${M_PI} ${-M_PI/4} 0"/>
+    </xacro:generic_camera>
 </robot>

Commit message: changed angle

File: jsk_mbzirc_tasks/urdf/quadrotor_with_hokyo30lx_and_downward_cam.urdf.xacro (robot description, xacro)
@@ -20,6 +20,6 @@
     <!-- side facing camera -->
     <xacro:generic_camera name="side_cam" parent="base_link" ros_topic="camera/image" cam_info_topic="camera/camera_info"
-			    update_rate="20" res_x="640" res_y="480" image_format="L8" hfov="100">
-      <origin xyz="-0.4 0.0 -0.0" rpy="${M_PI} ${-M_PI/4} 0"/>
+                          update_rate="20" res_x="640" res_y="480" image_format="L8" hfov="100">
+      <origin xyz="-0.4 0.0 -0.0" rpy="${M_PI} ${M_PI*0.75} 0"/>
     </xacro:generic_camera>
 </robot>
