Commit message: give a specific name for uav, called "hawk"

File: jsk_mbzirc_tasks/urdf/hawk.urdf.xacro (robot description, xacro)
@@ -14,5 +14,5 @@
       <origin xyz="0 0 0" rpy="0 0 0" />
       <geometry>
-        <mesh filename="package://jsk_mbzirc_tasks/urdf/meshes/tarrot680_p.stl" scale=".0254 .0254 .0254"/> <!-- mm has bug, right now use inch from ST8 -->
+        <mesh filename="package://jsk_mbzirc_tasks/urdf/meshes/hawk.stl" scale=".0254 .0254 .0254"/> <!-- mm has bug, right now use inch from ST8 -->
         <cylinder radius=".295" length=".23"/>
       </geometry>
@@ -24,5 +24,5 @@
       <origin xyz="0 0 0" rpy="0 0 0" />
       <geometry>
-        <mesh filename="package://jsk_mbzirc_tasks/urdf/meshes/tarrot680_p.stl" scale=".0254 .0254 .0254"/> <!-- mm has bug, right now use inch from ST8 -->
+        <mesh filename="package://jsk_mbzirc_tasks/urdf/meshes/hawk.stl" scale=".0254 .0254 .0254"/> <!-- mm has bug, right now use inch from ST8 -->
       </geometry>
     </collision>
