Commit message: fix two problem: 1) Set the "gravity" flag to 0 in terms of truck model to prevent from sinking into the ground. The possible reason is that the api "SetLinkWorkPose()" is conflict with the dynamics of truck. 2) Change from robot_ekf_pos to fake_localization which is aimed to publish tf from ground truth odometry.

File: jsk_mbzirc_common/urdf/truck.urdf.xacro (robot description, xacro)
@@ -7,5 +7,5 @@
       <mass value="700" /> <!-- http://trucktorack.blog.fc2.com/blog-entry-252.html -->
       <origin xyz="0 0 0.595" rpy="0 0 0" />
-      <inertia ixx="250.0" ixy="0.0" ixz="0.0" iyy="300.0" iyz="0.0" izz="300.0" />
+      <inertia ixx="200.0" ixy="0.0" ixz="0.0" iyy="400.0" iyz="0.0" izz="500.0" />
     </inertial>
     <visual>
@@ -35,5 +35,5 @@
       <mass value="20" />
       <origin xyz="0 0 0" rpy="0 0 0" />
-      <inertia ixx="0.18" ixy="0.0" ixz="0.0" iyy="0.18" iyz="0.0" izz="0.3" />
+      <inertia ixx="0.78" ixy="0.0" ixz="0.0" iyy="0.78" iyz="0.0" izz="0.87" />
     </inertial>
     <visual>
@@ -62,5 +62,5 @@
       <mass value="20" />
       <origin xyz="0 0 0" rpy="0 0 0" />
-      <inertia ixx="0.18" ixy="0.0" ixz="0.0" iyy="0.18" iyz="0.0" izz="0.3" />
+      <inertia ixx="0.78" ixy="0.0" ixz="0.0" iyy="0.78" iyz="0.0" izz="0.87" />
     </inertial>
     <visual>
@@ -89,5 +89,5 @@
       <mass value="20" />
       <origin xyz="0 0 0" rpy="0 0 0" />
-      <inertia ixx="0.18" ixy="0.0" ixz="0.0" iyy="0.18" iyz="0.0" izz="0.3" />
+      <inertia ixx="0.78" ixy="0.0" ixz="0.0" iyy="0.78" iyz="0.0" izz="0.87" />
     </inertial>
     <visual>
@@ -116,5 +116,5 @@
       <mass value="20" />
       <origin xyz="0 0 0" rpy="0 0 0" />
-      <inertia ixx="0.18" ixy="0.0" ixz="0.0" iyy="0.18" iyz="0.0" izz="0.3" />
+      <inertia ixx="0.78" ixy="0.0" ixz="0.0" iyy="0.78" iyz="0.0" izz="0.87" />
     </inertial>
     <visual>
@@ -141,7 +141,7 @@
   <link name="heliport">
     <inertial>
-      <mass value="10" />
-      <origin xyz="0 0 0" rpy="0 0 0" />
-      <inertia ixx="1.5" ixy="0.0" ixz="0.0" iyy="1.5" iyz="0.0" izz="3.0" />
+      <mass value="5" />
+      <origin xyz="0 0 0" rpy="0 0 0" />
+      <inertia ixx="1.0" ixy="0.0" ixz="0.0" iyy="1.0" iyz="0.0" izz="2.0" />
     </inertial>
     <visual>
@@ -166,6 +166,5 @@
       <bodyName>base_link</bodyName>
       <topicName>odom</topicName>
-      <updateRate>30.0</updateRate>
-<gaussianNoise>0.00001</gaussianNoise>
+      <updateRate>50.0</updateRate>
     </plugin>
     <!-- truck trajectory + task1 rule -->
@@ -182,4 +181,11 @@
     <gravity>0</gravity>
   </gazebo>
+  <gazebo reference="heliport">
+    <mu1>100</mu1>
+    <mu2>50</mu2>
+    <kp>1e+13</kp>
+    <kd>1</kd>
+    <gravity>0</gravity>
+  </gazebo>
   <gazebo reference="front_left_tire">
     <mu1>100</mu1>
@@ -187,6 +193,6 @@
     <kp>1e+13</kp>
     <kd>1</kd>
-    <gravity>0</gravity>
-    <material>Gazebo/Black</material>
+    <material>Gazebo/Black</material>
+    <gravity>0</gravity>
   </gazebo>
   <gazebo reference="front_right_tire">
@@ -196,4 +202,5 @@
     <kd>1</kd>
     <material>Gazebo/Black</material>
+    <gravity>0</gravity>
   </gazebo>
   <gazebo reference="rear_left_tire">
@@ -203,4 +210,5 @@
     <kd>1</kd>
     <material>Gazebo/Black</material>
+    <gravity>0</gravity>
   </gazebo>
   <gazebo reference="rear_right_tire">
@@ -210,4 +218,5 @@
     <kd>1</kd>
     <material>Gazebo/Black</material>
+    <gravity>0</gravity>
   </gazebo>
 </robot>
